File: KiCAD/LED-Test-Board.kicad_sch (KiCad schematic)
At the start: 37 parts, among them U2 ULN2803A

Commit message: README変更、回路修正
Parts:
- C1: value (none) -> 10u
- D1: value (none) -> LED0
- D10: value (none) -> LED9
- D11: value (none) -> LED10
- D12: value (none) -> LED11
- D13: value (none) -> LED12
- D14: value (none) -> LED13
- D15: value (none) -> LED14
- D16: value (none) -> LED15
- D17: renamed from D?; value (none) -> LED16
- D18: renamed from D?; value (none) -> LED17
- D19: renamed from D?; value (none) -> LED18
- D2: value (none) -> LED1
- D20: renamed from D?; value (none) -> LED19
- D21: renamed from D?; value (none) -> LED20
- D22: renamed from D?; value (none) -> LED21
- D23: renamed from D?; value (none) -> LED22
- D24: renamed from D?; value (none) -> LED23
- D3: value (none) -> LED2
- D4: value (none) -> LED3
- D5: value (none) -> LED4
- D6: value (none) -> LED5
- D7: value (none) -> LED6
- D8: value (none) -> LED7
- D9: value (none) -> LED8
- J1: value (none) -> CON-A
- J2: value (none) -> CON-B
- RN1: value (none) -> 10k; footprint (none) -> Resistor_THT:R_Array_SIP9
- RN3: value (none) -> 1k
- U1: value (none) -> ULN2803A
- gave numbers to parts that had none: 3
Connections:
- net PA0: now also RN1.9 (R8), U1.8 (I8); no longer RN1.2 (R1), U1.1 (I1)
- net PA1: now also RN1.8 (R7), U1.7 (I7); no longer RN1.3 (R2), U1.2 (I2)
- net PA2: now also RN1.7 (R6), U1.6 (I6); no longer RN1.4 (R3), U1.3 (I3)
- net PA3: now also RN1.6 (R5), U1.5 (I5); no longer RN1.5 (R4), U1.4 (I4)
- net PA4: now also RN1.5 (R4), U1.4 (I4); no longer RN1.6 (R5), U1.5 (I5)
- net PA5: now also RN1.4 (R3), U1.3 (I3); no longer RN1.7 (R6), U1.6 (I6)
- net PA6: now also RN1.3 (R2), U1.2 (I2); no longer RN1.8 (R7), U1.7 (I7)
- net PA7: now also RN1.2 (R1), U1.1 (I1); no longer RN1.9 (R8), U1.8 (I8)
- net PB0: now also RN2.9 (R8), U2.8 (I8); no longer RN2.2 (R1), U2.1 (I1)
- net PB1: now also RN2.8 (R7), U2.7 (I7); no longer RN2.3 (R2), U2.2 (I2)
- net PB2: now also RN2.7 (R6), U2.6 (I6); no longer RN2.4 (R3), U2.3 (I3)
- net PB3: now also RN2.6 (R5), U2.5 (I5); no longer RN2.5 (R4), U2.4 (I4)
- net PB4: now also RN2.5 (R4), U2.4 (I4); no longer RN2.6 (R5), U2.5 (I5)
- net PB5: now also RN2.4 (R3), U2.3 (I3); no longer RN2.7 (R6), U2.6 (I6)
- net PB6: now also RN2.3 (R2), U2.2 (I2); no longer RN2.8 (R7), U2.7 (I7)
- net PB7: now also RN2.2 (R1), U2.1 (I1); no longer RN2.9 (R8), U2.8 (I8)
- net PC0: now also RN5.9 (R8), U3.8 (I8); no longer RN5.2 (R1), U3.1 (I1)
- net PC1: now also RN5.8 (R7), U3.7 (I7); no longer RN5.3 (R2), U3.2 (I2)
- net PC2: now also RN5.7 (R6), U3.6 (I6); no longer RN5.4 (R3), U3.3 (I3)
- net PC3: now also RN5.6 (R5), U3.5 (I5); no longer RN5.5 (R4), U3.4 (I4)
- net PC4: now also RN5.5 (R4), U3.4 (I4); no longer RN5.6 (R5), U3.5 (I5)
- net PC5: now also RN5.4 (R3), U3.3 (I3); no longer RN5.7 (R6), U3.6 (I6)
- net PC6: now also RN5.3 (R2), U3.2 (I2); no longer RN5.8 (R7), U3.7 (I7)
- net PC7: now also RN5.2 (R1), U3.1 (I1); no longer RN5.9 (R8), U3.8 (I8)
